File: hananMiniPcb/hananMiniPcb.kicad_sch (KiCad schematic)
At the start: 23 parts, among them J2 Conn_02x04_Top_Bottom, U1 MCP4901

Commit message: hananMiniPcb v2.0: pads arcade en columna, RC en Vref + 100n en Vdd, pads D1, rótulo de versión
- J2 header 1x08 -> huella ODS:Hanan_PadsArcade_1x08_Pares (8 pads 3.5 mm en columna,
  pares señal/GND, orden blanco/rosa/amarillo/verde), zona GND a toda la placa, M3 como huellas.
- Contorno 150x75 reconstruido del gerber JLC P169.
- R6 1k + C2 10u en Vref (net VREF), C3 100n en Vdd del MCP4901; +5C reruteado.
- Pads de D1 1.25x1.8 (anillo 0.175); stubs/vías colgadas de Pin_4 borrados.
- Title block + silk 'hananMiniPcb ${REVISION} ${ISSUE_DATE}' en F y B.
- docs/revision-electronica-mini.md: revisión eléctrica y alcance de la rev.

Co-Authored-By: Claude Fable 5.1 <noreply@anthropic.com>
Claude-Session: https://claude.ai/code/session_018KSRbDX7mTqiibDixEKAXu
Parts:
- added C2: 10uF, Capacitor_THT:CP_Radial_D4.0mm_P2.00mm, symbol BD1-rescue-2020-02-22-22-49-19:CP1
- added C3: 100nF, Capacitor_THT:C_Disc_D5.0mm_W2.5mm_P5.00mm, symbol Device:C
- added R6: 1k, Resistor_THT:R_Axial_DIN0207_L6.3mm_D2.5mm_P7.62mm_Horizontal, symbol BD1-rescue-2020-02-22-22-49-19:R
Connections:
- net +5C: now also C3.1, R6.1; no longer U1.6 (Vref)
- net GND: now also C2.2, C3.2
- new net VREF: C2.1, R6.2, U1.6 (Vref)
Other:
- note added: "MODS v2.0 2026-10-07: RC en Vref + 100n en Vdd"
- company: (none) -> Oficina de Sonido
- title: (none) -> hananMiniPcb
