File: hardware/hananClasicaPcb/hananClasicaPcb.kicad_sch (KiCad schematic)
At the start: 23 parts, among them J2 Conn_02x04_Top_Bottom, U1 MCP4901

Commit message: Reorganización: repo en la raíz de hanan-cumbia, hardware/ firmware/ docs/, PCB clásica v2.0
- Raíz del repo = hanan-cumbia/ (antes hanan26/); webflasher/ y hananFabrica/ siguen en la raíz
  (GitHub Pages no cambia).
- hardware/hananMiniPcb (limpio: solo pro/sch/pcb/bom) y hardware/hananClasicaPcb (nuevo, v2.0 con
  RC en Vref, 100n en Vdd, pads D1, rótulo de versión; sch = el del Mini + J1/D2).
- firmware/hanan26Taller, firmware/tests/*, firmware/legacy/HTRCMB_10.
- docs/: revisión eléctrica, capas EasyEDA, SVG de calados del panel Mini.
- Fuera del repo: Placa_2021, HTR_2023, hanan25, códigos/audios viejos y backups → 3-archivo/hanan-cumbia-historico.

Co-Authored-By: Claude Fable 5.1 <noreply@anthropic.com>
Claude-Session: https://claude.ai/code/session_018KSRbDX7mTqiibDixEKAXu
Parts:
- added C2: 10uF, Capacitor_THT:CP_Radial_D4.0mm_P2.00mm, symbol BD1-rescue-2020-02-22-22-49-19:CP1
- added C3: 100nF, Capacitor_THT:C_Disc_D5.0mm_W2.5mm_P5.00mm, symbol Device:C
- added D2: DIODE, Diode_THT:D_A-405_P7.62mm_Horizontal, symbol Device:D
- added J1: Jack-DC, OdeS:jack_dc_solder, symbol Connector:Barrel_Jack_Switch
- added R6: 1k, Resistor_THT:R_Axial_DIN0207_L6.3mm_D2.5mm_P7.62mm_Horizontal, symbol BD1-rescue-2020-02-22-22-49-19:R
Connections:
- net +5C: now also C3.1, R6.1; no longer U1.6 (Vref)
- net +9V: now also D2.1 (K)
- net GND: now also C2.2, C3.2, J1.2
- new net VIN_JACK: D2.2 (A), J1.1
- new net VREF: C2.1, R6.2, U1.6 (Vref)
- no-connect marks 0 -> 1
Other:
- note added: "MODS v2.0 2026-10-07: RC en Vref + 100n en Vdd"
- company: (none) -> Oficina de Sonido
- title: (none) -> hananClasicaPcb

Commit message: hananClasicaPcb v2.0: J2 header -> columna de pads arcade compacta (ODS), gerber regenerado
Co-Authored-By: Claude Fable 5.1 <noreply@anthropic.com>
Claude-Session: https://claude.ai/code/session_018KSRbDX7mTqiibDixEKAXu
Parts:
- J2: footprint Connector_PinHeader_2.00mm:PinHeader_1x08_P2.00mm_Vertical -> ODS:Hanan_PadsArcade_1x08_Pares_Compacto
Changed lines of the file:
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@@
 			)
 		)
-		(property "Footprint" "Connector_PinHeader_2.00mm:PinHeader_1x08_P2.00mm_Vertical"
+		(property "Footprint" "ODS:Hanan_PadsArcade_1x08_Pares_Compacto"
 			(at 248.92 72.39 0)
 			(effects
