File: hardware/hananMiniPcb/hananMiniPcb.kicad_sch (KiCad schematic)
At the start: 26 parts, among them J2 Conn_02x04_Top_Bottom, U1 MCP4901

Commit message: hananClasicaPcb v2.0: J2 header -> columna de pads arcade compacta (ODS), gerber regenerado
Co-Authored-By: Claude Fable 5.1 <noreply@anthropic.com>
Claude-Session: https://claude.ai/code/session_018KSRbDX7mTqiibDixEKAXu
Parts:
- J2: footprint Connector_PinHeader_2.00mm:PinHeader_1x08_P2.00mm_Vertical -> ODS:Hanan_PadsArcade_1x08_Pares
Changed lines of the file:
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@@
 			)
 		)
-		(property "Footprint" "Connector_PinHeader_2.00mm:PinHeader_1x08_P2.00mm_Vertical"
+		(property "Footprint" "ODS:Hanan_PadsArcade_1x08_Pares"
 			(at 248.92 72.39 0)
 			(effects
